File: Current_Inputs.kicad_sch (KiCad schematic)
At the start: 16 parts, among them J4 ANALOG VOLTAGE INPUTS, U7 D3V3XA4B10LP

Commit message: added remaining pages. BOM and refinement is all thats left
Parts:
- removed C10, C11, C12, C13, C14, C9: 0.1uF, symbol Device:C
- removed C6: 4.7nF, symbol Device:C
- removed C7: 1uF, symbol Device:C
- removed C8: 10uF, symbol Device:C
- removed J4: ANALOG VOLTAGE INPUTS, symbol Connector_Generic:Conn_01x05
- removed R17, R18, R19, R20: 1k, symbol Device:R
- removed U6: (no value), Package_QFP:TQFP-64_10x10mm_P0.5mm, symbol Custom_DT1042-04SO-7:ADS1261
- removed U7: D3V3XA4B10LP, Package_DFN_QFN:Diodes_UDFN-10_1x2.5mm_P0.5mm, symbol Power_Protection:D3V3XA4B10LP
- added C20, C23, C25, C26, C27: 0.1uF, symbol Device:C
- added C21: 4.7nF, symbol Device:C
- added C22: 1uF, symbol Device:C
- added C24: 10uF, symbol Device:C
- added J6: CURRENT INPUTS, symbol Connector_Generic:Conn_01x06
- added R23, R24, R25: 47R, symbol Device:R
- added R26, R27, R28, R29, R30, R31: 1k, symbol Device:R
- added U10: (no value), Package_QFP:TQFP-64_10x10mm_P0.5mm, symbol Custom_DT1042-04SO-7:ADS1261
- added U9: D3V3XA4B10LP, Package_DFN_QFN:Diodes_UDFN-10_1x2.5mm_P0.5mm, symbol Power_Protection:D3V3XA4B10LP
Connections:
- net +3.3V: now also C23.1, U10.17 (DVDD)
- net +5V: now also C20.2, U10.4 (AVDD)
- net GND: now also C20.1, C22.2, C23.2, C24.2, J6.2 (Pin_2), J6.4 (Pin_4), J6.6 (Pin_6), R23.2, R24.2, R25.2, R27.1, R29.1, R31.1, U10.1 (AINCOM), U10.16 (DGND), U10.18 (CLKIN), U10.33 (AVSS_EP), U10.5 (AVSS), U9.3 (VSS), U9.8 (VSS)
- net SPI_PICO: now also U10.12 (DIN)
- net SPI_POCI: now also U10.14 (DOUT/DRDY)
- net SPI_SCK: now also U10.11 (SCLK)
- new net: C24.1, U10.6 (REFOUT)
- new net: C22.1, U10.15 (BYPASS)
- new net: C26.1, R28.2, U10.30 (AIN2)
- new net: C26.2, R29.2, U10.29 (AIN3)
- new net: J6.5 (Pin_5), R25.1, R30.1, U9.4
- new net: C27.1, R30.2, U10.28 (AIN4)
- new net: J6.1 (Pin_1), R23.1, R26.1, U9.1
- new net: J6.3 (Pin_3), R24.1, R28.1, U9.2
- new net: C27.2, R31.2, U10.27 (AIN5)
- new net: C21.1, U10.2 (CAPP)
- new net: C21.2, U10.3 (CAPN)
- new net: C25.2, R27.2, U10.31 (AIN1)
- new net: C25.1, R26.2, U10.32 (AIN0)
- new net ADC2_CS: U10.10 (CS)
- new net ADC2_DRDY: U10.13 (DRDY)
- new net ADC2_PWDN: U10.7 (PWDN)
- new net ADC2_RESET: U10.8 (RESET)
- new net ADC2_START: U10.9 (START)
- no-connect marks 8 -> 9
Other:
- title: Analog Voltage Inputs -> Current Inputs

Commit message: Added a few comments in blue text
Other:
- note added: "Missing current amplifers"
Changed lines of the file:
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@@
 		(company "Slap DAQ")
+	)
+	(text "Missing current amplifers"
+		(exclude_from_sim no)
+		(at 73.66 59.436 0)
+		(effects
+			(font
+				(size 1.27 1.27)
+			)
+		)
 	)
 	(junction

Commit message: finished schematic draft 1
Parts:
- removed R29, R30, R31: 1k, symbol Device:R
- removed U10: (no value), Package_QFP:TQFP-64_10x10mm_P0.5mm, symbol Custom_DT1042-04SO-7:ADS1261
- added C39, C41, C42, C43: 0.1uF, symbol Device:C
- added C40: 1uF, symbol Device:C
- added U10, U16, U6: INA181, Package_TO_SOT_SMD:SOT-23-6, symbol Amplifier_Current:INA181
- added U14: ADS1261, Package_DFN_QFN:QFN-32-1EP_5x5mm_P0.5mm_EP3.45x3.45mm, symbol Custom_ADS1261:ADS1261
- added U15: REF3333, Package_TO_SOT_SMD:SOT-23, symbol Custom_REF3333:REF3333
- C21: value 4.7nF -> 4.7nF C0G
- J6: footprint (none) -> TerminalBlock_Phoenix:TerminalBlock_Phoenix_MKDS-1,5-6-5.08_1x06_P5.08mm_Horizontal; MPN (none) -> 1715763; Manufacturer (none) -> Phoenix Contact
- R23, R24, R25: value 47R -> 3R
- U9: MPN (none) -> D3V3XA4B10LP-7; Manufacturer (none) -> Diodes Incorporated
Connections:
- net +3.3V: now also U14.17 (DVDD)
- net +5V: now also C39.1, C41.1, C42.1, C43.1, U10.6 (V+), U14.4 (AVDD), U15.1 (IN), U16.6 (V+), U6.6 (V+)
- net ADC2_CS: now also U14.10 (CS)
- net ADC2_DRDY: now also U14.13 (DRDY)
- net ADC2_PWDN: now also U14.7 (PWDN)
- net ADC2_RESET: now also U14.8 (RESET)
- net ADC2_START: now also U14.9 (START)
- net GND: now also C25.2, C26.2, C27.2, J6.3 (Pin_3), R24.1, U9.2, C39.2, C40.2, C41.2, C42.2, C43.2, U10.2 (GND), U10.5 (REF), U14.1 (AINCOM), U14.16 (DGND), U14.18 (CLKIN), U14.30 (AIN2), U14.33 (AVSS_EP), U14.5 (AVSS), U15.3 (GND), U16.2 (GND), U16.3 (+), U16.4 (-), U16.5 (REF), U6.2 (GND), U6.3 (+), U6.4 (-), U6.5 (REF); no longer J6.4 (Pin_4), R24.2, R27.1
- net SPI_PICO: now also U14.12 (DIN)
- net SPI_POCI: now also U14.14 (DOUT/DRDY)
- net SPI_SCK: now also U14.11 (SCLK)
- net at C24.1: now also U14.6 (REFOUT)
- net at C22.1: now also U14.15 (BYPASS)
- net at C26.1: now also R27.2, U14.25 (AIN7); no longer R28.2
- net at C27.1: now also R28.2, U14.24 (AIN8)
- net at J6.1 (Pin_1), R23.1, U9.1: no longer R26.1
- net at C21.1: now also U14.2 (CAPP)
- net at C21.2: now also U14.3 (CAPN)
- net at C25.1, R26.2: now also U14.26 (AIN6)
- new net: R27.1, U10.1
- new net: J6.4 (Pin_4), R24.2, U10.3 (+), U10.4 (-)
- new net: C40.1, U14.32 (AIN0), U15.2 (OUT)
- new net: R28.1, U16.1
- new net: R26.1, U6.1
- no-connect marks 9 -> 10
Other:
- note removed: "Missing current amplifers"
- title: Current Inputs -> Current Input
- moved on the sheet: C20, C21, C22, C23, C24, C25, C26, C27, J6, R23, R24, R25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

Commit message: Fixed some issues and renamed project
Parts:
- U14: symbol Custom_ADS1261:ADS1261 -> Custom_Symbols:ADS1261
- U15: symbol Custom_REF3333:REF3333 -> Custom_Symbols:REF3333
Connections:
- net GND: no longer U14.16 (DGND)
