File: Analog_Voltage_Inputs.kicad_sch (KiCad schematic)
At the start: 16 parts, among them J4 ANALOG VOLTAGE INPUTS, U7 D3V3XA4B10LP

Commit message: Added a few comments in blue text
Other:
- note added: "C6 needs to be a C0G type MLCC"
- note added: "Missing voltage reference IC (1 for each ADC)"
Changed lines of the file:
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@@
 		(company "Slap DAQ")
+	)
+	(text "Missing voltage reference IC (1 for each ADC)"
+		(exclude_from_sim no)
+		(at 205.232 71.12 0)
+		(effects
+			(font
+				(size 1.27 1.27)
+			)
+		)
+	)
+	(text "C6 needs to be a C0G type MLCC"
+		(exclude_from_sim no)
+		(at 137.922 131.572 0)
+		(effects
+			(font
+				(size 1.27 1.27)
+			)
+		)
 	)
 	(junction

Commit message: finished schematic draft 1
Parts:
- removed U6: (no value), Package_QFP:TQFP-64_10x10mm_P0.5mm, symbol Custom_DT1042-04SO-7:ADS1261
- added C37: 0.1uF, symbol Device:C
- added C38: 1uF, symbol Device:C
- added U12: REF3333, Package_TO_SOT_SMD:SOT-23, symbol Custom_REF3333:REF3333
- added U13: ADS1261, Package_DFN_QFN:QFN-32-1EP_5x5mm_P0.5mm_EP3.45x3.45mm, symbol Custom_ADS1261:ADS1261
- C6: value 4.7nF -> 4.7nF C0G
- J4: footprint (none) -> TerminalBlock_Phoenix:TerminalBlock_Phoenix_MKDS-1,5-5-5.08_1x05_P5.08mm_Horizontal; MPN (none) -> 1715750; Manufacturer (none) -> Phoenix Contact
- U7: MPN (none) -> D3V3XA4B10LP-7; Manufacturer (none) -> Diodes Incorporated
Connections:
- net +3.3V: now also U13.17 (DVDD)
- net +5V: now also C37.1, U12.1 (IN), U13.4 (AVDD)
- net ADC1_CS: now also U13.10 (CS)
- net ADC1_DRDY: now also U13.13 (DRDY)
- net ADC1_PWDN: now also U13.7 (PWDN)
- net ADC1_RESET: now also U13.8 (RESET)
- net ADC1_START: now also U13.9 (START)
- net DIFF_IN_N: now also U13.27 (AIN5)
- net DIFF_IN_P: now also U13.28 (AIN4)
- net GND: now also C11.2, C12.2, C13.2, C14.2, C37.2, C38.2, U12.3 (GND), U13.1 (AINCOM), U13.16 (DGND), U13.18 (CLKIN), U13.30 (AIN2), U13.33 (AVSS_EP), U13.5 (AVSS); no longer C11.1, C12.1, C13.1, C14.1
- net SPI_PICO: now also U13.12 (DIN)
- net SPI_POCI: now also U13.14 (DOUT/DRDY)
- net SPI_SCK: now also U13.11 (SCLK)
- net at R17.2: now also C11.1, U13.26 (AIN6); no longer C11.2
- net at C6.1: now also U13.2 (CAPP)
- net at C6.2: now also U13.3 (CAPN)
- net at R18.2: now also C12.1, U13.25 (AIN7); no longer C12.2
- net at C7.1: now also U13.15 (BYPASS)
- net at R20.2: now also C14.1, U13.23 (AIN9); no longer C14.2
- net at R19.2: now also C13.1, U13.24 (AIN8); no longer C13.2
- net at C8.1: now also U13.6 (REFOUT)
- new net: C38.1, U12.2 (OUT), U13.32 (AIN0)
- no-connect marks 8 -> 6
Other:
- note removed: "C6 needs to be a C0G type MLCC"
- note removed: "Missing voltage reference IC (1 for each ADC)"
- moved on the sheet: C10, C11, C12, C13, C14, C7, C8, C9, J4, R17, R18, R19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

Commit message: Fixed some issues and renamed project
Parts:
- U12: symbol Custom_REF3333:REF3333 -> Custom_Symbols:REF3333
- U13: symbol Custom_ADS1261:ADS1261 -> Custom_Symbols:ADS1261
Connections:
- net GND: no longer U13.16 (DGND)
Changed lines of the file:
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@@
 		)
 		(instances
-			(project "capstoneKicad"
+			(project "slapdaq-board"
 				(path "/13b31ec5-9d44-45c3-b3e5-a18c48e5f516/6cb30bb6-2ed8-4e19-9b9a-43b34b8df240"
 					(reference "#PWR034")
@@
 		)
 		(instances
-			(project "capstoneKicad"
+			(project "slapdaq-board"
 				(path "/13b31ec5-9d44-45c3-b3e5-a18c48e5f516/6cb30bb6-2ed8-4e19-9b9a-43b34b8df240"
 					(reference "R17")
@@
 		)
 		(instances
-			(project "capstoneKicad"
+			(project "slapdaq-board"
 				(path "/13b31ec5-9d44-45c3-b3e5-a18c48e5f516/6cb30bb6-2ed8-4e19-9b9a-43b34b8df240"
 					(reference "#PWR028")
@@
 		)
 		(instances
-			(project "capstoneKicad"
+			(project "slapdaq-board"
 				(path "/13b31ec5-9d44-45c3-b3e5-a18c48e5f516/6cb30bb6-2ed8-4e19-9b9a-43b34b8df240"
 					(reference "#PWR027")
@@
 		)
 		(instances
-			(project "capstoneKicad"
+			(project "slapdaq-board"
 				(path "/13b31ec5-9d44-45c3-b3e5-a18c48e5f516/6cb30bb6-2ed8-4e19-9b9a-43b34b8df240"
 					(reference "C6")
@@
 		)
 		(instances
-			(project "capstoneKicad"
+			(project "slapdaq-board"
 				(path "/13b31ec5-9d44-45c3-b3e5-a18c48e5f516/6cb30bb6-2ed8-4e19-9b9a-43b34b8df240"
 					(reference "#PWR070")
@@
 		)
 		(instances
-			(project "capstoneKicad"
+			(project "slapdaq-board"
 				(path "/13b31ec5-9d44-45c3-b3e5-a18c48e5f516/6cb30bb6-2ed8-4e19-9b9a-43b34b8df240"
 					(reference "#PWR026")
@@
 		)
 		(instances
-			(project "capstoneKicad"
+			(project "slapdaq-board"
 				(path "/13b31ec5-9d44-45c3-b3e5-a18c48e5f516/6cb30bb6-2ed8-4e19-9b9a-43b34b8df240"
 					(reference "R18")
@@
 		)
 		(instances
-			(project "capstoneKicad"
+			(project "slapdaq-board"
 				(path "/13b31ec5-9d44-45c3-b3e5-a18c48e5f516/6cb30bb6-2ed8-4e19-9b9a-43b34b8df240"
 					(reference "C12")
@@
 		)
 		(instances
-			(project "capstoneKicad"
+			(project "slapdaq-board"
 				(path "/13b31ec5-9d44-45c3-b3e5-a18c48e5f516/6cb30bb6-2ed8-4e19-9b9a-43b34b8df240"
 					(reference "#PWR037")
@@
 		)
 		(instances
-			(project "capstoneKicad"
+			(project "slapdaq-board"
 				(path "/13b31ec5-9d44-45c3-b3e5-a18c48e5f516/6cb30bb6-2ed8-4e19-9b9a-43b34b8df240"
 					(reference "#PWR023")
@@
 		)
 		(instances
-			(project "capstoneKicad"
+			(project "slapdaq-board"
 				(path "/13b31ec5-9d44-45c3-b3e5-a18c48e5f516/6cb30bb6-2ed8-4e19-9b9a-43b34b8df240"
 					(reference "C38")
@@
 		)
 		(instances
-			(project "capstoneKicad"
+			(project "slapdaq-board"
 				(path "/13b31ec5-9d44-45c3-b3e5-a18c48e5f516/6cb30bb6-2ed8-4e19-9b9a-43b34b8df240"
 					(reference "#PWR013")
@@
 		)
 		(instances
-			(project "capstoneKicad"
+			(project "slapdaq-board"
 				(path "/13b31ec5-9d44-45c3-b3e5-a18c48e5f516/6cb30bb6-2ed8-4e19-9b9a-43b34b8df240"
 					(reference "C13")
@@
 		)
 		(instances
-			(project "capstoneKicad"
+			(project "slapdaq-board"
 				(path "/13b31ec5-9d44-45c3-b3e5-a18c48e5f516/6cb30bb6-2ed8-4e19-9b9a-43b34b8df240"
 					(reference "#PWR071")
@@
 	)
 	(symbol
-		(lib_id "Custom_REF3333:REF3333")
+		(lib_id "Custom_Symbols:REF3333")
 		(at 109.22 74.93 0)
 		(unit 1)
@@
 		)
 		(instances
-			(project "capstoneKicad"
+			(project "slapdaq-board"
 				(path "/13b31ec5-9d44-45c3-b3e5-a18c48e5f516/6cb30bb6-2ed8-4e19-9b9a-43b34b8df240"
 					(reference "U12")
@@
 		)
 		(instances
-			(project "capstoneKicad"
+			(project "slapdaq-board"
 				(path "/13b31ec5-9d44-45c3-b3e5-a18c48e5f516/6cb30bb6-2ed8-4e19-9b9a-43b34b8df240"
 					(reference "#PWR033")
@@
 		)
 		(instances
-			(project "capstoneKicad"
+			(project "slapdaq-board"
 				(path "/13b31ec5-9d44-45c3-b3e5-a18c48e5f516/6cb30bb6-2ed8-4e19-9b9a-43b34b8df240"
 					(reference "C37")
@@
 		)
 		(instances
-			(project "capstoneKicad"
+			(project "slapdaq-board"
 				(path "/13b31ec5-9d44-45c3-b3e5-a18c48e5f516/6cb30bb6-2ed8-4e19-9b9a-43b34b8df240"
 					(reference "C7")
@@
 		)
 		(instances
-			(project "capstoneKicad"
+			(project "slapdaq-board"
 				(path "/13b31ec5-9d44-45c3-b3e5-a18c48e5f516/6cb30bb6-2ed8-4e19-9b9a-43b34b8df240"
 					(reference "C10")
@@
 		)
 		(instances
-			(project "capstoneKicad"
+			(project "slapdaq-board"
 				(path "/13b31ec5-9d44-45c3-b3e5-a18c48e5f516/6cb30bb6-2ed8-4e19-9b9a-43b34b8df240"
 					(reference "#PWR029")
@@
 		)
 		(instances
-			(project "capstoneKicad"
+			(project "slapdaq-board"
 				(path "/13b31ec5-9d44-45c3-b3e5-a18c48e5f516/6cb30bb6-2ed8-4e19-9b9a-43b34b8df240"
 					(reference "#PWR024")
@@
 		)
 		(instances
-			(project "capstoneKicad"
+			(project "slapdaq-board"
 				(path "/13b31ec5-9d44-45c3-b3e5-a18c48e5f516/6cb30bb6-2ed8-4e19-9b9a-43b34b8df240"
 					(reference "U7")
@@
 		)
 		(instances
-			(project "capstoneKicad"
+			(project "slapdaq-board"
 				(path "/13b31ec5-9d44-45c3-b3e5-a18c48e5f516/6cb30bb6-2ed8-4e19-9b9a-43b34b8df240"
 					(reference "C8")
@@
 		)
 		(instances
-			(project "capstoneKicad"
+			(project "slapdaq-board"
 				(path "/13b31ec5-9d44-45c3-b3e5-a18c48e5f516/6cb30bb6-2ed8-4e19-9b9a-43b34b8df240"
 					(reference "C11")
@@
 		)
 		(instances
-			(project "capstoneKicad"
+			(project "slapdaq-board"
 				(path "/13b31ec5-9d44-45c3-b3e5-a18c48e5f516/6cb30bb6-2ed8-4e19-9b9a-43b34b8df240"
 					(reference "#PWR025")
@@
 		)
 		(instances
-			(project "capstoneKicad"
+			(project "slapdaq-board"
 				(path "/13b31ec5-9d44-45c3-b3e5-a18c48e5f516/6cb30bb6-2ed8-4e19-9b9a-43b34b8df240"
 					(reference "#PWR031")
@@
 		)
 		(instances
-			(project "capstoneKicad"
+			(project "slapdaq-board"
 				(path "/13b31ec5-9d44-45c3-b3e5-a18c48e5f516/6cb30bb6-2ed8-4e19-9b9a-43b34b8df240"
 					(reference "#PWR072")
@@
 		)
 		(instances
-			(project "capstoneKicad"
+			(project "slapdaq-board"
 				(path "/13b31ec5-9d44-45c3-b3e5-a18c48e5f516/6cb30bb6-2ed8-4e19-9b9a-43b34b8df240"
 					(reference "#PWR069")
@@
 		)
 		(instances
-			(project "capstoneKicad"
+			(project "slapdaq-board"
 				(path "/13b31ec5-9d44-45c3-b3e5-a18c48e5f516/6cb30bb6-2ed8-4e19-9b9a-43b34b8df240"
 					(reference "C14")
@@
 		)
 		(instances
-			(project "capstoneKicad"
+			(project "slapdaq-board"
 				(path "/13b31ec5-9d44-45c3-b3e5-a18c48e5f516/6cb30bb6-2ed8-4e19-9b9a-43b34b8df240"
 					(reference "#PWR022")
@@
 		)
 		(instances
-			(project "capstoneKicad"
+			(project "slapdaq-board"
 				(path "/13b31ec5-9d44-45c3-b3e5-a18c48e5f516/6cb30bb6-2ed8-4e19-9b9a-43b34b8df240"
 					(reference "J4")
@@
 		)
 		(instances
-			(project "capstoneKicad"
+			(project "slapdaq-board"
 				(path "/13b31ec5-9d44-45c3-b3e5-a18c48e5f516/6cb30bb6-2ed8-4e19-9b9a-43b34b8df240"
 					(reference "R20")
@@
 		)
 		(instances
-			(project "capstoneKicad"
+			(project "slapdaq-board"
 				(path "/13b31ec5-9d44-45c3-b3e5-a18c48e5f516/6cb30bb6-2ed8-4e19-9b9a-43b34b8df240"
 					(reference "#PWR035")
@@
 		)
 		(instances
-			(project "capstoneKicad"
+			(project "slapdaq-board"
 				(path "/13b31ec5-9d44-45c3-b3e5-a18c48e5f516/6cb30bb6-2ed8-4e19-9b9a-43b34b8df240"
 					(reference "#PWR032")
@@
 		)
 		(instances
-			(project "capstoneKicad"
+			(project "slapdaq-board"
 				(path "/13b31ec5-9d44-45c3-b3e5-a18c48e5f516/6cb30bb6-2ed8-4e19-9b9a-43b34b8df240"
 					(reference "#PWR014")
@@
 		)
 		(instances
-			(project "capstoneKicad"
+			(project "slapdaq-board"
 				(path "/13b31ec5-9d44-45c3-b3e5-a18c48e5f516/6cb30bb6-2ed8-4e19-9b9a-43b34b8df240"
 					(reference "R19")
@@
 		)
 		(instances
-			(project "capstoneKicad"
+			(project "slapdaq-board"
 				(path "/13b31ec5-9d44-45c3-b3e5-a18c48e5f516/6cb30bb6-2ed8-4e19-9b9a-43b34b8df240"
 					(reference "#PWR036")
@@
 		)
 		(instances
-			(project "capstoneKicad"
+			(project "slapdaq-board"
 				(path "/13b31ec5-9d44-45c3-b3e5-a18c48e5f516/6cb30bb6-2ed8-4e19-9b9a-43b34b8df240"
 					(reference "C9")
@@
 	)
 	(symbol
-		(lib_id "Custom_ADS1261:ADS1261")
+		(lib_id "Custom_Symbols:ADS1261")
 		(at 167.64 99.06 0)
 		(unit 1)
@@
 		(in_pos_files yes)
 		(dnp no)
-		(fields_autoplaced yes)
 		(property "Reference" "U13"
-			(at 173.5933 78.74 0)
+			(at 173.736 78.994 0)
 			(show_name no)
 			(do_not_autoplace no)
@@
 		)
 		(property "Value" "ADS1261"
-			(at 167.64 99.06 0)
+			(at 163.322 99.314 0)
 			(show_name no)
 			(do_not_autoplace no)
@@
 					(size 1.27 1.27)
 				)
+				(justify left)
 			)
 		)
@@
 		)
 		(instances
-			(project "capstoneKicad"
+			(project "slapdaq-board"
 				(path "/13b31ec5-9d44-45c3-b3e5-a18c48e5f516/6cb30bb6-2ed8-4e19-9b9a-43b34b8df240"
 					(reference "U13")
@@
 		)
 		(instances
-			(project "capstoneKicad"
+			(project "slapdaq-board"
 				(path "/13b31ec5-9d44-45c3-b3e5-a18c48e5f516/6cb30bb6-2ed8-4e19-9b9a-43b34b8df240"
 					(reference "#PWR073")

Commit message: "combined analog voltage and differential voltage sheets
Parts:
- added C44: 0.1uF, symbol Device:C
- added J8: DIFFERENTIAL VOLTAGE INPUT, TerminalBlock_Phoenix:TerminalBlock_Phoenix_MKDS-1,5-3-5.08_1x03_P5.08mm_Horizontal, symbol Connector_Generic:Conn_01x03
- added R29, R30: 1k, symbol Device:R
- added U17: D3V3XA4B10LP, Package_DFN_QFN:Diodes_UDFN-10_1x2.5mm_P0.5mm, symbol Power_Protection:D3V3XA4B10LP
Connections:
- net GND: now also J8.3 (Pin_3), U17.3 (VSS), U17.8 (VSS)
- net DIFF_IN_N: no longer names the net of U13.27 (AIN5)
- net DIFF_IN_N: now also C44.2, R30.2
- net DIFF_IN_P: no longer names the net of U13.28 (AIN4)
- net DIFF_IN_P: now also C44.1, R29.2
- new net: J8.1 (Pin_1), R29.1, U17.1
- new net: J8.2 (Pin_2), R30.1, U17.2
- no-connect marks 6 -> 12
Other:
- title: Analog Voltage Inputs -> ADC
- moved on the sheet: C37, C38, U12
