File: MCU_DIO.kicad_sch (KiCad schematic)
At the start: 14 parts, among them J2 USB-C, J3 DIGITAL_IO_3V3, U3 ESP32-S3

Commit message: changed sheet names
Other:
- title: ESP32 / Digital I/O -> MCU
Changed lines of the file:
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@@
 	(paper "A")
 	(title_block
-		(title "ESP32 / Digital I/O")
+		(title "MCU")
 		(date "2026-09-08")
 		(rev "1")

Commit message: changed net labels to global labels
Other:
- moved on the sheet: J3
Changed lines of the file:
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@@
 	(text "SPI MOSI = D\nSPI MISO = Q"
 		(exclude_from_sim no)
-		(at 96.012 121.412 0)
+		(at 89.662 121.412 0)
 		(effects
 			(font
@@
 	(text "Add TVS arrays if needed"
 		(exclude_from_sim no)
-		(at 84.074 89.662 0)
+		(at 77.724 89.662 0)
 		(effects
 			(font
@@
 	(wire
 		(pts
-			(xy 111.76 114.3) (xy 120.65 114.3)
+			(xy 116.84 111.76) (xy 120.65 111.76)
 		)
 		(stroke
@@
 	(wire
 		(pts
+			(xy 116.84 114.3) (xy 120.65 114.3)
+		)
+		(stroke
+			(width 0)
+			(type default)
+		)
+	)
+	(wire
+		(pts
 			(xy 179.07 118.11) (xy 177.8 118.11)
 		)
@@
 	(wire
 		(pts
-			(xy 92.71 104.14) (xy 120.65 104.14)
+			(xy 86.36 104.14) (xy 120.65 104.14)
 		)
 		(stroke
@@
 	(wire
 		(pts
-			(xy 105.41 127) (xy 105.41 109.22)
+			(xy 97.79 127) (xy 97.79 109.22)
 		)
 		(stroke
@@
 	(wire
 		(pts
-			(xy 120.65 127) (xy 105.41 127)
-		)
-		(stroke
-			(width 0)
-			(type default)
-		)
-	)
-	(wire
-		(pts
-			(xy 92.71 96.52) (xy 120.65 96.52)
-		)
-		(stroke
-			(width 0)
-			(type default)
-		)
-	)
-	(wire
-		(pts
-			(xy 111.76 119.38) (xy 120.65 119.38)
+			(xy 116.84 106.68) (xy 120.65 106.68)
+		)
+		(stroke
+			(width 0)
+			(type default)
+		)
+	)
+	(wire
+		(pts
+			(xy 120.65 127) (xy 97.79 127)
+		)
+		(stroke
+			(width 0)
+			(type default)
+		)
+	)
+	(wire
+		(pts
+			(xy 86.36 96.52) (xy 120.65 96.52)
 		)
 		(stroke
@@
 	(wire
 		(pts
-			(xy 111.76 106.68) (xy 120.65 106.68)
-		)
-		(stroke
-			(width 0)
-			(type default)
-		)
-	)
-	(wire
-		(pts
-			(xy 92.71 111.76) (xy 96.52 111.76)
+			(xy 86.36 111.76) (xy 90.17 111.76)
 		)
 		(stroke
@@
 	(wire
 		(pts
-			(xy 107.95 124.46) (xy 120.65 124.46)
+			(xy 100.33 124.46) (xy 120.65 124.46)
 		)
 		(stroke
@@
 	(wire
 		(pts
-			(xy 107.95 106.68) (xy 92.71 106.68)
+			(xy 100.33 106.68) (xy 86.36 106.68)
 		)
 		(stroke
@@
 	(wire
 		(pts
-			(xy 107.95 124.46) (xy 107.95 106.68)
+			(xy 100.33 124.46) (xy 100.33 106.68)
 		)
 		(stroke
@@
 	(wire
 		(pts
-			(xy 111.76 116.84) (xy 120.65 116.84)
-		)
-		(stroke
-			(width 0)
-			(type default)
-		)
-	)
-	(wire
-		(pts
 			(xy 204.47 113.03) (xy 208.28 113.03)
 		)
@@
 	(wire
 		(pts
+			(xy 116.84 119.38) (xy 120.65 119.38)
+		)
+		(stroke
+			(width 0)
+			(type default)
+		)
+	)
+	(wire
+		(pts
 			(xy 200.66 91.44) (xy 204.47 91.44)
 		)
@@
 	(wire
 		(pts
-			(xy 111.76 111.76) (xy 120.65 111.76)
-		)
-		(stroke
-			(width 0)
-			(type default)
-		)
-	)
-	(wire
-		(pts
 			(xy 172.72 83.82) (xy 172.72 113.03)
 		)
@@
 	(wire
 		(pts
+			(xy 116.84 116.84) (xy 120.65 116.84)
+		)
+		(stroke
+			(width 0)
+			(type default)
+		)
+	)
+	(wire
+		(pts
 			(xy 151.13 86.36) (xy 154.94 86.36)
 		)
@@
 	(wire
 		(pts
-			(xy 92.71 99.06) (xy 120.65 99.06)
+			(xy 86.36 99.06) (xy 120.65 99.06)
 		)
 		(stroke
@@
 	(wire
 		(pts
-			(xy 105.41 109.22) (xy 92.71 109.22)
+			(xy 97.79 109.22) (xy 86.36 109.22)
 		)
 		(stroke
@@
 	(wire
 		(pts
-			(xy 92.71 101.6) (xy 120.65 101.6)
+			(xy 86.36 101.6) (xy 120.65 101.6)
 		)
 		(stroke
@@
 	(wire
 		(pts
-			(xy 92.71 114.3) (xy 96.52 114.3)
+			(xy 86.36 114.3) (xy 90.17 114.3)
 		)
 		(stroke
@@
 	)
 	(label "DIO3"
-		(at 96.52 101.6 0)
-		(effects
-			(font
-				(size 1.27 1.27)
-			)
-			(justify left bottom)
-		)
-	)
-	(label "SPI_D"
-		(at 111.76 114.3 0)
+		(at 90.17 101.6 0)
 		(effects
 			(font
@@
 	)
 	(label "DIO1"
-		(at 96.52 96.52 0)
+		(at 90.17 96.52 0)
 		(effects
 			(font
@@
 	)
 	(label "DIO7"
-		(at 96.52 111.76 0)
+		(at 90.17 111.76 0)
 		(effects
 			(font
@@
 	)
 	(label "DIO2"
-		(at 96.52 99.06 0)
+		(at 90.17 99.06 0)
 		(effects
 			(font
@@
 	)
 	(label "DIO5"
-		(at 96.52 106.68 0)
+		(at 90.17 106.68 0)
 		(effects
 			(font
@@
 		)
 	)
-	(label "CS1_THR"
-		(at 111.76 106.68 0)
+	(label "DIO4"
+		(at 90.17 104.14 0)
 		(effects
 			(font
@@
 		)
 	)
-	(label "DIO4"
-		(at 96.52 104.14 0)
+	(label "DIO8"
+		(at 90.17 114.3 0)
 		(effects
 			(font
@@
 		)
 	)
-	(label "DIO8"
-		(at 96.52 114.3 0)
+	(label "DIO6"
+		(at 90.17 109.22 0)
 		(effects
 			(font
@@
 		)
 	)
-	(label "DIO6"
-		(at 96.52 109.22 0)
+	(global_label "CS0_ADC"
+		(shape input)
+		(at 116.84 111.76 180)
+		(fields_autoplaced yes)
 		(effects
 			(font
 				(size 1.27 1.27)
 			)
-			(justify left bottom)
-		)
-	)
-	(label "SPI_CLK"
-		(at 111.76 116.84 0)
+			(justify right)
+		)
+		(property "Intersheetrefs" "${INTERSHEET_REFS}"
+			(at 105.5696 111.76 0)
+			(hide yes)
+			(show_name no)
+			(do_not_autoplace no)
+			(effects
+				(font
+					(size 1.27 1.27)
+				)
+				(justify right)
+			)
+		)
+	)
+	(global_label "SPI_D"
+		(shape input)
+		(at 116.84 114.3 180)
+		(fields_autoplaced yes)
 		(effects
 			(font
 				(size 1.27 1.27)
 			)
-			(justify left bottom)
-		)
-	)
-	(label "SPI_Q"
-		(at 111.76 119.38 0)
+			(justify right)
+		)
+		(property "Intersheetrefs" "${INTERSHEET_REFS}"
+			(at 108.5329 114.3 0)
+			(hide yes)
+			(show_name no)
+			(do_not_autoplace no)
+			(effects
+				(font
+					(size 1.27 1.27)
+				)
+				(justify right)
+			)
+		)
+	)
+	(global_label "CS1_THR"
+		(shape input)
+		(at 116.84 106.68 180)
+		(fields_autoplaced yes)
 		(effects
 			(font
 				(size 1.27 1.27)
 			)
-			(justify left bottom)
-		)
-	)
-	(label "CS0_ADC"
-		(at 111.76 111.76 0)
+			(justify right)
+		)
+		(property "Intersheetrefs" "${INTERSHEET_REFS}"
+			(at 105.6301 106.68 0)
+			(hide yes)
+			(show_name no)
+			(do_not_autoplace no)
+			(effects
+				(font
+					(size 1.27 1.27)
+				)
+				(justify right)
+			)
+		)
+	)
+	(global_label "SPI_Q"
+		(shape input)
+		(at 116.84 119.38 180)
+		(fields_autoplaced yes)
 		(effects
 			(font
 				(size 1.27 1.27)
 			)
-			(justify left bottom)
+			(justify right)
+		)
+		(property "Intersheetrefs" "${INTERSHEET_REFS}"
+			(at 108.4724 119.38 0)
+			(hide yes)
+			(show_name no)
+			(do_not_autoplace no)
+			(effects
+				(font
+					(size 1.27 1.27)
+				)
+				(justify right)
+			)
+		)
+	)
+	(global_label "SPI_CLK"
+		(shape input)
+		(at 116.84 116.84 180)
+		(fields_autoplaced yes)
+		(effects
+			(font
+				(size 1.27 1.27)
+			)
+			(justify right)
+		)
+		(property "Intersheetrefs" "${INTERSHEET_REFS}"
+			(at 106.2348 116.84 0)
+			(hide yes)
+			(show_name no)
+			(do_not_autoplace no)
+			(effects
+				(font
+					(size 1.27 1.27)
+				)
+				(justify right)
+			)
 		)
 	)
@@
 	(symbol
 		(lib_id "Connector_Generic:Conn_01x08")
-		(at 87.63 104.14 0)
+		(at 81.28 104.14 0)
 		(mirror y)
 		(unit 1)
@@
 		(dnp no)
 		(property "Reference" "J3"
-			(at 88.646 93.726 0)
+			(at 82.296 93.726 0)
 			(show_name no)
 			(do_not_autoplace no)
@@
 		)
 		(property "Value" "DIGITAL_IO_3V3"
-			(at 91.694 128.27 0)
+			(at 85.344 128.27 0)
 			(hide yes)
 			(show_name no)
@@
 		)
 		(property "Footprint" "TerminalBlock_Phoenix:TerminalBlock_Phoenix_MKDS-1,5-8-5.08_1x08_P5.08mm_Horizontal"
-			(at 87.63 104.14 0)
+			(at 81.28 104.14 0)
 			(hide yes)
 			(show_name no)
@@
 		)
 		(property "Datasheet" ""
-			(at 87.63 104.14 0)
+			(at 81.28 104.14 0)
 			(hide yes)
 			(show_name no)
@@
 		)
 		(property "Description" "Generic connector, single row, 01x08, script generated (kicad-library-utils/schlib/autogen/connector/)"
-			(at 87.63 104.14 0)
+			(at 81.28 104.14 0)
 			(hide yes)
 			(show_name no)
@@
 		)
 		(property "Manufacturer" "Phoenix Contact"
-			(at 87.63 104.14 0)
+			(at 81.28 104.14 0)
 			(hide yes)
 			(show_name no)
@@
 		)
 		(property "MPN" "1729128"
-			(at 87.63 104.14 0)
-			(hide yes)
-			(show_name no)
+			(at 81.28 104.14 0)
+			(hide yes)
+			(show_name no)

Commit message: added gnd to inputs
Parts:
- removed J3: DIGITAL_IO_3V3, TerminalBlock_Phoenix:TerminalBlock_Phoenix_MKDS-1,5-8-5.08_1x08_P5.08mm_Horizontal, symbol Connector_Generic:Conn_01x08
- added J5: DIGITAL IO INPUTS, symbol Connector_Generic:Conn_01x09
Connections:
- net DIO1: now also J5.1 (Pin_1)
- net DIO2: now also J5.2 (Pin_2)
- net DIO3: now also J5.3 (Pin_3)
- net DIO4: now also J5.4 (Pin_4)
- net DIO5: now also J5.5 (Pin_5)
- net DIO6: now also J5.6 (Pin_6)
- net DIO7: now also J5.7 (Pin_7)
- net DIO8: now also J5.8 (Pin_8)
- net GND: now also J5.9 (Pin_9)
Changed lines of the file:
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@@
 	(text "SPI MOSI = D\nSPI MISO = Q"
 		(exclude_from_sim no)
-		(at 89.662 121.412 0)
+		(at 60.452 117.602 0)
 		(effects
 			(font
@@
 	(text "Add TVS arrays if needed"
 		(exclude_from_sim no)
-		(at 77.724 89.662 0)
+		(at 66.04 114.046 0)
 		(effects
 			(font
@@
 	(wire
 		(pts
+			(xy 86.36 116.84) (xy 90.17 116.84)
+		)
+		(stroke
+			(width 0)
+			(type default)
+		)
+	)
+	(wire
+		(pts
 			(xy 233.68 123.19) (xy 233.68 121.92)
 		)
@@
 	)
 	(symbol
+		(lib_id "Connector_Generic:Conn_01x09")
+		(at 81.28 106.68 0)
+		(mirror y)
+		(unit 1)
+		(body_style 1)
+		(exclude_from_sim no)
+		(in_bom yes)
+		(on_board yes)
+		(in_pos_files yes)
+		(dnp no)
+		(fields_autoplaced yes)
+		(property "Reference" "J5"
+			(at 81.28 90.17 0)
+			(show_name no)
+			(do_not_autoplace no)
+			(effects
+				(font
+					(size 1.27 1.27)
+				)
+			)
+		)
+		(property "Value" "DIGITAL IO INPUTS"
+			(at 81.28 92.71 0)
+			(show_name no)
+			(do_not_autoplace no)
+			(effects
+				(font
+					(size 1.27 1.27)
+				)
+			)
+		)
+		(property "Footprint" ""
+			(at 81.28 106.68 0)
+			(hide yes)
+			(show_name no)
+			(do_not_autoplace no)
+			(effects
+				(font
+					(size 1.27 1.27)
+				)
+			)
+		)
+		(property "Datasheet" ""
+			(at 81.28 106.68 0)
+			(hide yes)
+			(show_name no)
+			(do_not_autoplace no)
+			(effects
+				(font
+					(size 1.27 1.27)
+				)
+			)
+		)
+		(property "Description" "Generic connector, single row, 01x09, script generated (kicad-library-utils/schlib/autogen/connector/)"
+			(at 81.28 106.68 0)
+			(hide yes)
+			(show_name no)
+			(do_not_autoplace no)
+			(effects
+				(font
+					(size 1.27 1.27)
+				)
+			)
+		)
+		(pin "1"
+		)
+		(pin "5"
+		)
+		(pin "6"
+		)
+		(pin "2"
+		)
+		(pin "7"
+		)
+		(pin "9"
+		)
+		(pin "3"
+		)
+		(pin "4"
+		)
+		(pin "8"
+		)
+		(instances
+			(project "slapdaq-board"
+				(path "/13b31ec5-9d44-45c3-b3e5-a18c48e5f516/f3b0adef-1da3-4963-a2de-79e7f8ea7f57"
+					(reference "J5")
+					(unit 1)
+				)
+			)
+		)
+	)
+	(symbol
 		(lib_id "power:GND")
 		(at 106.68 80.01 0)
@@
 	)
 	(symbol
-		(lib_id "Connector_Generic:Conn_01x08")
-		(at 81.28 104.14 0)
-		(mirror y)
-		(unit 1)
-		(body_style 1)
-		(exclude_from_sim no)
-		(in_bom yes)
-		(on_board yes)
-		(in_pos_files yes)
-		(dnp no)
-		(property "Reference" "J3"
-			(at 82.296 93.726 0)
-			(show_name no)
-			(do_not_autoplace no)
-			(effects
-				(font
-					(size 1.27 1.27)
-				)
-				(justify left)
-			)
-		)
-		(property "Value" "DIGITAL_IO_3V3"
-			(at 85.344 128.27 0)
-			(hide yes)
-			(show_name no)
-			(do_not_autoplace no)
-			(effects
-				(font
-					(size 1.27 1.27)
-				)
-				(justify left)
-			)
-		)
-		(property "Footprint" "TerminalBlock_Phoenix:TerminalBlock_Phoenix_MKDS-1,5-8-5.08_1x08_P5.08mm_Horizontal"
-			(at 81.28 104.14 0)
-			(hide yes)
-			(show_name no)
-			(do_not_autoplace no)
-			(effects
-				(font
-					(size 1.27 1.27)
-				)
-			)
-		)
-		(property "Datasheet" ""
-			(at 81.28 104.14 0)
-			(hide yes)
-			(show_name no)
-			(do_not_autoplace no)
-			(effects
-				(font
-					(size 1.27 1.27)
-				)
-			)
-		)
-		(property "Description" "Generic connector, single row, 01x08, script generated (kicad-library-utils/schlib/autogen/connector/)"
-			(at 81.28 104.14 0)
-			(hide yes)
-			(show_name no)
-			(do_not_autoplace no)
-			(effects
-				(font
-					(size 1.27 1.27)
-				)
-			)
-		)
-		(property "Manufacturer" "Phoenix Contact"
-			(at 81.28 104.14 0)
-			(hide yes)
-			(show_name no)
-			(do_not_autoplace no)
-			(effects
-				(font
-					(size 1.27 1.27)
-				)
-			)
-		)
-		(property "MPN" "1729128"
-			(at 81.28 104.14 0)
-			(hide yes)
-			(show_name no)
-			(do_not_autoplace no)
-			(effects
-				(font
-					(size 1.27 1.27)
-				)
-			)
-		)
-		(pin "1"
-		)
-		(pin "4"
-		)
-		(pin "3"
-		)
-		(pin "8"
-		)
-		(pin "6"
-		)
-		(pin "5"
-		)
-		(pin "2"
-		)
-		(pin "7"
-		)
-		(instances
-			(project "slapdaq-board"
-				(path "/13b31ec5-9d44-45c3-b3e5-a18c48e5f516/f3b0adef-1da3-4963-a2de-79e7f8ea7f57"
-					(reference "J3")
-					(unit 1)
-				)
-			)
-		)
-	)
-	(symbol
 		(lib_id "Device:LED")
 		(at 121.92 168.91 90)
@@
 					(unit 1)
 				)
+			)
+		)
+	)
+	(symbol
+		(lib_id "power:GND")
+		(at 90.17 116.84 0)
+		(unit 1)
+		(body_style 1)
+		(exclude_from_sim no)
+		(in_bom yes)
+		(on_board yes)
+		(in_pos_files yes)
+		(dnp no)
+		(fields_autoplaced yes)
+		(property "Reference" "#PWR019"
+			(at 90.17 123.19 0)
+			(hide yes)
+			(show_name no)
+			(do_not_autoplace no)
+			(effects
+				(font
+					(size 1.27 1.27)
+				)
+			)
+		)
+		(property "Value" "GND"
+			(at 90.17 121.92 0)
+			(show_name no)
+			(do_not_autoplace no)
+			(effects
+				(font
+					(size 1.27 1.27)
+				)
+			)
+		)
+		(property "Footprint" ""
+			(at 90.17 116.84 0)
+			(hide yes)
+			(show_name no)
+			(do_not_autoplace no)
+			(effects
+				(font
+					(size 1.27 1.27)
+				)
+			)
+		)
+		(property "Datasheet" ""
+			(at 90.17 116.84 0)
+			(hide yes)
+			(show_name no)
+			(do_not_autoplace no)
+			(effects
+				(font
+					(size 1.27 1.27)
+				)
+			)
+		)
+		(property "Description" "Power symbol creates a global label with name \"GND\" , ground"
+			(at 90.17 116.84 0)
+			(hide yes)
+			(show_name no)
+			(do_not_autoplace no)
+			(effects
+				(font
+					(size 1.27 1.27)
+				)
+			)
+		)
+		(pin "1"
+		)
+		(instances
+			(project "slapdaq-board"
+				(path "/13b31ec5-9d44-45c3-b3e5-a18c48e5f516/f3b0adef-1da3-4963-a2de-79e7f8ea7f57"
+					(reference "#PWR019")
+					(unit 1)
+				)
