File: slapdaq-board.kicad_sch (KiCad schematic)
At the start: 21 parts, among them J1 12-24V POWER IN, U1 LMR51430 - 5V REG, U2 LMR51430 - 3.3V REG

Commit message: "combined analog voltage and differential voltage sheets
Other:
- sheet Analog_Voltage_Inputs renamed ADC
- removed sheet Differential_Voltage_Input
Changed lines of the file:
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@@
 			(color 0 0 0 0)
 		)
-		(property "Sheetname" "Analog_Voltage_Inputs"
+		(property "Sheetname" "ADC"
 			(at 184.15 86.9184 0)
 			(show_name no)
@@
 				)
 			)
-		)
-	)
-	(sheet
-		(at 184.15 113.03)
-		(size 31.75 16.51)
-		(exclude_from_sim no)
-		(in_bom yes)
-		(on_board yes)
-		(dnp no)
-		(fields_autoplaced yes)
-		(stroke
-			(width 0.1524)
-			(type solid)
-		)
-		(fill
-			(color 0 0 0 0)
-		)
-		(property "Sheetname" "Differential_Voltage_Input"
-			(at 184.15 112.3184 0)
-			(show_name no)
-			(do_not_autoplace no)
-			(effects
-				(font
-					(size 1.27 1.27)
-				)
-				(justify left bottom)
-			)
-		)
-		(property "Sheetfile" "Differential_Voltage_Input.kicad_sch"
-			(at 184.15 130.1246 0)
-			(show_name no)
-			(do_not_autoplace no)
-			(effects
-				(font
-					(size 1.27 1.27)
-				)
-				(justify left top)
-			)
-		)
-		(instances
-			(project "slapdaq-board"
-				(path "/13b31ec5-9d44-45c3-b3e5-a18c48e5f516"
-					(page "4")
-				)
-			)

Commit message: Grayson changes 9/11/26
Parts:
- removed C1: 10uF, 50V, symbol Device:C
- removed C2, C32: 0.1uF, symbol Device:C
- removed C30, C35: 4.7uF, 50V, symbol Device:C
- removed C31, C36: 0.1uF, 50V, symbol Device:C
- removed C33, C34: 22uF, 25V, symbol Device:C
- removed R35, R37: 100k, symbol Device:R
- removed R36: 13.7k, symbol Device:R
- removed R38: 22.1k, symbol Device:R
- removed U1: LMR51430 - 5V REG, Package_TO_SOT_SMD:SOT-23-6, symbol Regulator_Switching:LMR51430
- removed U2: LMR51430 - 3.3V REG, Package_TO_SOT_SMD:SOT-23-6, symbol Regulator_Switching:LMR51430
- added C1, C15, C30: 100u, symbol Device:C_Polarized
- added C2: 68u, symbol Device:C_Polarized
- added D4, D5: D_Schottky, symbol Device:D_Schottky
- added U1: LM2675M-3.3, Package_SO:SOIC-8_3.9x4.9mm_P1.27mm, symbol Regulator_Switching:LM2675M-3.3
- added U2: LM2675M-5, Package_SO:SOIC-8_3.9x4.9mm_P1.27mm, symbol Regulator_Switching:LM2675M-5
- C29, C3: value 22uF, 25V -> 0.01u
- L1: value 6.8uH -> 47u; footprint Package_TO_SOT_SMD:SOT-23-6 -> (none)
- L2: value 5.6uH -> 68u; footprint Package_TO_SOT_SMD:SOT-23-6 -> (none)
Connections:
- net +3.3V: now also L1.2, C2.1; no longer C3.1, L2.2
- net +5V: now also L2.2, C30.1; no longer C29.1, L1.2
- net GND: now also C1.2, C15.2, C2.2, C30.2, D4.2 (A), D5.2 (A), U1.6 (GND), U2.6 (GND); no longer C29.2, C3.2
- net at L2.1: now also C29.2, D5.1 (K), U2.4 (FB), U2.8 (VSW)
- net at L1.1: now also C3.2, D4.1 (K), U1.4 (FB), U1.8 (VSW)
- net VIN_12V_24V: no longer names the net of F1.2
- net VIN_12V_24V: now also C1.1, C15.1, U1.5 (ON/~{OFF}), U1.7 (VIN), U2.5 (ON/~{OFF}), U2.7 (VIN)
- new net: C3.1, U1.1 (CB)
- new net: C29.1, U2.1 (CB)

Commit message: 9/13/2026 schematic work
Other:
- sheet ESP32_Digital_IO renamed MCU_DIO
- sheet Thermocouple_Input renamed Thermocouple
- removed sheet Current_Inputs
- sheet ADC: file Analog_Voltage_Inputs.kicad_sch -> ADC.kicad_sch
- sheet MCU_DIO: file ESP32_Digital_IO.kicad_sch -> MCU_DIO.kicad_sch
- sheet Thermocouple: file Thermocouple_Input.kicad_sch -> Thermocouple.kicad_sch
Changed lines of the file:
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@@
 	)
 	(sheet
-		(at 184.15 87.63)
+		(at 198.12 78.74)
 		(size 31.75 16.51)
 		(exclude_from_sim no)
@@
 		)
 		(property "Sheetname" "ADC"
-			(at 184.15 86.9184 0)
+			(at 198.12 78.0284 0)
 			(show_name no)
 			(do_not_autoplace no)
@@
 			)
 		)
-		(property "Sheetfile" "Analog_Voltage_Inputs.kicad_sch"
-			(at 184.15 104.7246 0)
+		(property "Sheetfile" "ADC.kicad_sch"
+			(at 198.12 95.8346 0)
 			(show_name no)
 			(do_not_autoplace no)
@@
 	)
 	(sheet
-		(at 227.33 76.2)
+		(at 198.12 101.6)
 		(size 31.75 16.51)
 		(exclude_from_sim no)
@@
 			(color 0 0 0 0)
 		)
-		(property "Sheetname" "Current_Inputs"
-			(at 227.33 75.4884 0)
+		(property "Sheetname" "Thermocouple"
+			(at 198.12 100.8884 0)
 			(show_name no)
 			(do_not_autoplace no)
@@
 			)
 		)
-		(property "Sheetfile" "Current_Inputs.kicad_sch"
-			(at 227.33 93.2946 0)
+		(property "Sheetfile" "Thermocouple.kicad_sch"
+			(at 198.12 118.6946 0)
 			(show_name no)
 			(do_not_autoplace no)
@@
 			(project "slapdaq-board"
 				(path "/13b31ec5-9d44-45c3-b3e5-a18c48e5f516"
-					(page "5")
+					(page "4")
 				)
 			)
@@
 	)
 	(sheet
-		(at 226.06 102.87)
+		(at 198.12 55.88)
 		(size 31.75 16.51)
 		(exclude_from_sim no)
@@
 			(color 0 0 0 0)
 		)
-		(property "Sheetname" "Thermocouple_Input"
-			(at 226.06 102.1584 0)
+		(property "Sheetname" "MCU_DIO"
+			(at 198.12 55.1684 0)
 			(show_name no)
 			(do_not_autoplace no)
@@
 			)
 		)
-		(property "Sheetfile" "Thermocouple_Input.kicad_sch"
-			(at 226.06 119.9646 0)
+		(property "Sheetfile" "MCU_DIO.kicad_sch"
+			(at 198.12 72.9746 0)
 			(show_name no)
 			(do_not_autoplace no)
-			(effects
-				(font
-					(size 1.27 1.27)
-				)
-				(justify left top)
-			)
-		)
-		(instances
-			(project "slapdaq-board"
-				(path "/13b31ec5-9d44-45c3-b3e5-a18c48e5f516"
-					(page "6")
-				)
-			)
-		)
-	)
-	(sheet
-		(at 184.15 60.96)
-		(size 31.75 16.51)
-		(exclude_from_sim no)
-		(in_bom yes)
-		(on_board yes)
-		(dnp no)
-		(fields_autoplaced yes)
-		(stroke
-			(width 0.1524)
-			(type solid)
-		)
-		(fill
-			(color 0 0 0 0)
-		)
-		(property "Sheetname" "ESP32_Digital_IO"
-			(at 184.15 60.2484 0)
-			(show_name no)
-			(do_not_autoplace no)
-			(effects
-				(font
-					(size 1.27 1.27)
-				)
-				(justify left bottom)
-			)
-		)
-		(property "Sheetfile" "ESP32_Digital_IO.kicad_sch"
-			(at 184.15 78.0546 0)
-			(show_name no)
-			(do_not_autoplace no)

Commit message: changed sheet names
Other:
- sheet MCU_DIO renamed MCU
- title: System/Power -> Power
Changed lines of the file:
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@@
 	(paper "A")
 	(title_block
-		(title "System/Power")
+		(title "Power")
 		(date "2026-09-08")
 		(rev "1")
@@
 			(color 0 0 0 0)
 		)
-		(property "Sheetname" "MCU_DIO"
+		(property "Sheetname" "MCU"
 			(at 198.12 55.1684 0)
 			(show_name no)

Commit message: 9/18/2026 schematic work
Other:
- sheet MCU: file MCU_DIO.kicad_sch -> MCU.kicad_sch
- note added: "For Grayson: Connect Vbus to the input of the 3.3 V regulator (and the +5V net?) I think that will allow the entire device to work with only USB power. Use schottky diodes."
Changed lines of the file:
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@@
 		(comment 3 "ESET")
+	)
+	(text "For Grayson: Connect Vbus to the input of the 3.3 V regulator (and the +5V net?)\nI think that will allow the entire device to work with only USB power.\nUse schottky diodes."
+		(exclude_from_sim no)
+		(at 148.59 91.44 0)
+		(effects
+			(font
+				(size 1.27 1.27)
+			)
+		)
 	)
 	(junction
@@
 			(width 0)
 			(type default)
+		)
+	)
+	(global_label "Vbus"
+		(shape input)
+		(at 135.89 100.33 0)
+		(fields_autoplaced yes)
+		(effects
+			(font
+				(size 1.27 1.27)
+			)
+			(justify left)
+		)
+		(property "Intersheetrefs" "${INTERSHEET_REFS}"
+			(at 143.2899 100.33 0)
+			(hide yes)
+			(show_name no)
+			(do_not_autoplace no)
+			(effects
+				(font
+					(size 1.27 1.27)
+				)
+				(justify left)
+			)
 		)
 	)
@@
 			)
 		)
+		(property "Mouser Link" ""
+			(at 63.5 109.22 0)
+			(hide yes)
+			(show_name no)
+			(do_not_autoplace no)
+			(effects
+				(font
+					(size 1.27 1.27)
+				)
+			)
+		)
 		(pin "2"
 		)
@@
 			)
 		)
+		(property "Mouser Link" ""
+			(at 120.65 113.03 0)
+			(hide yes)
+			(show_name no)
+			(do_not_autoplace no)
+			(effects
+				(font
+					(size 1.27 1.27)
+				)
+			)
+		)
 		(pin "2"
 		)
@@
 			)
 		)
+		(property "Mouser Link" ""
+			(at 85.09 63.5 0)
+			(hide yes)
+			(show_name no)
+			(do_not_autoplace no)
+			(effects
+				(font
+					(size 1.27 1.27)
+				)
+			)
+		)
 		(pin "3"
 		)
@@
 			)
 		)
+		(property "Mouser Link" ""
+			(at 85.09 101.6 0)
+			(hide yes)
+			(show_name no)
+			(do_not_autoplace no)
+			(effects
+				(font
+					(size 1.27 1.27)
+				)
+			)
+		)
 		(pin "8"
 		)
@@
 			)
 		)
+		(property "Mouser Link" ""
+			(at 113.03 68.58 90)
+			(hide yes)
+			(show_name no)
+			(do_not_autoplace no)
+			(effects
+				(font
+					(size 1.27 1.27)
+				)
+			)
+		)
 		(pin "2"
 		)
@@
 			)
 		)
+		(property "Mouser Link" ""
+			(at 113.03 106.68 90)
+			(hide yes)
+			(show_name no)
+			(do_not_autoplace no)
+			(effects
+				(font
+					(size 1.27 1.27)
+				)
+			)
+		)
 		(pin "2"
 		)
@@
 			)
 		)
+		(property "Mouser Link" ""
+			(at 104.14 73.66 90)
+			(hide yes)
+			(show_name no)
+			(do_not_autoplace no)
+			(effects
+				(font
+					(size 1.27 1.27)
+				)
+			)
+		)
 		(pin "1"
 		)
@@
 		(property "Description" "Unpolarized capacitor"
 			(at 102.87 63.5 0)
+			(hide yes)
+			(show_name no)
+			(do_not_autoplace no)
+			(effects
+				(font
+					(size 1.27 1.27)
+				)
+			)
+		)
+		(property "Mouser Link" ""
+			(at 102.87 63.5 90)
 			(hide yes)
 			(show_name no)
@@
 			)
 		)
+		(property "Mouser Link" ""
+			(at 102.87 101.6 90)
+			(hide yes)
+			(show_name no)
+			(do_not_autoplace no)
+			(effects
+				(font
+					(size 1.27 1.27)
+				)
+			)
+		)
 		(pin "1"
 		)
@@
 		)
 		(property "MPN" "595D686X9010C2T"
+			(at 120.65 76.2 0)
+			(hide yes)
+			(show_name no)
+			(do_not_autoplace no)
+			(effects
+				(font
+					(size 1.27 1.27)
+				)
+			)
+		)
+		(property "Mouser Link" ""
 			(at 120.65 76.2 0)
 			(hide yes)
@@
 			)
 		)
+		(property "Mouser Link" ""
+			(at 40.64 58.42 0)
+			(hide yes)
+			(show_name no)
+			(do_not_autoplace no)
+			(effects
+				(font
+					(size 1.27 1.27)
+				)
+			)
+		)
 		(pin "1"
 		)
@@
 			)
 		)
+		(property "Mouser Link" ""
+			(at 63.5 72.39 0)
+			(hide yes)
+			(show_name no)
+			(do_not_autoplace no)
+			(effects
+				(font
+					(size 1.27 1.27)
+				)
+			)
+		)
 		(pin "2"
 		)
@@
 			)
 		)
+		(property "Mouser Link" ""
+			(at 52.07 58.42 0)
+			(hide yes)
+			(show_name no)
+			(do_not_autoplace no)
+			(effects
+				(font
+					(size 1.27 1.27)
+				)
+			)
+		)
 		(pin "1"
 		)
@@
 			)
 		)
+		(property "Mouser Link" ""
+			(at 104.14 113.03 90)
+			(hide yes)
+			(show_name no)
+			(do_not_autoplace no)
+			(effects
+				(font
+					(size 1.27 1.27)
+				)
+			)
+		)
 		(pin "1"
 		)
@@
 			)
 		)
-		(property "Sheetfile" "MCU_DIO.kicad_sch"
+		(property "Sheetfile" "MCU.kicad_sch"
 			(at 198.12 72.9746 0)
 			(show_name no)

Commit message: removed grounds from inputs
Parts:
- renumbered C15 to C2, C29 to C4, C2 to C5, C30 to C6, D4 to D1, D5 to D2
Changed lines of the file:
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@@
 		(dnp no)
 		(fields_autoplaced yes)
-		(property "Reference" "#PWR030"
+		(property "Reference" "#PWR07"
 			(at 104.14 124.46 0)
 			(hide yes)
@@
 			(project "slapdaq-board"
 				(path "/13b31ec5-9d44-45c3-b3e5-a18c48e5f516"
-					(reference "#PWR030")
+					(reference "#PWR07")
 					(unit 1)
 				)
@@
 		(dnp no)
 		(fields_autoplaced yes)
-		(property "Reference" "#PWR03"
+		(property "Reference" "#PWR09"
 			(at 120.65 87.63 0)
 			(hide yes)
@@
 			(project "slapdaq-board"
 				(path "/13b31ec5-9d44-45c3-b3e5-a18c48e5f516"
-					(reference "#PWR03")
+					(reference "#PWR09")
 					(unit 1)
 				)
@@
 		(dnp no)
 		(fields_autoplaced yes)
-		(property "Reference" "C15"
+		(property "Reference" "C2"
 			(at 67.31 107.0609 0)
 			(show_name no)
@@
 			(project "slapdaq-board"
 				(path "/13b31ec5-9d44-45c3-b3e5-a18c48e5f516"
-					(reference "C15")
+					(reference "C2")
 					(unit 1)
 				)
@@
 		(dnp no)
 		(fields_autoplaced yes)
-		(property "Reference" "#PWR018"
+		(property "Reference" "#PWR05"
 			(at 85.09 120.65 0)
 			(hide yes)
@@
 			(project "slapdaq-board"
 				(path "/13b31ec5-9d44-45c3-b3e5-a18c48e5f516"
-					(reference "#PWR018")
+					(reference "#PWR05")
 					(unit 1)
 				)
@@
 		(dnp no)
 		(fields_autoplaced yes)
-		(property "Reference" "#PWR07"
+		(property "Reference" "#PWR03"
 			(at 63.5 120.65 0)
 			(hide yes)
@@
 			(project "slapdaq-board"
 				(path "/13b31ec5-9d44-45c3-b3e5-a18c48e5f516"
-					(reference "#PWR07")
+					(reference "#PWR03")
 					(unit 1)
 				)
@@
 		(dnp no)
 		(fields_autoplaced yes)
-		(property "Reference" "#PWR04"
+		(property "Reference" "#PWR02"
 			(at 63.5 83.82 0)
 			(hide yes)
@@
 			(project "slapdaq-board"
 				(path "/13b31ec5-9d44-45c3-b3e5-a18c48e5f516"
-					(reference "#PWR04")
+					(reference "#PWR02")
 					(unit 1)
 				)
@@
 		(dnp no)
 		(fields_autoplaced yes)
-		(property "Reference" "C30"
+		(property "Reference" "C6"
 			(at 124.46 110.8709 0)
 			(show_name no)
@@
 			(project "slapdaq-board"
 				(path "/13b31ec5-9d44-45c3-b3e5-a18c48e5f516"
-					(reference "C30")
+					(reference "C6")
 					(unit 1)
 				)
@@
 		(dnp no)
 		(fields_autoplaced yes)
-		(property "Reference" "#PWR045"
+		(property "Reference" "#PWR010"
 			(at 120.65 104.14 0)
 			(hide yes)
@@
 			(project "slapdaq-board"
 				(path "/13b31ec5-9d44-45c3-b3e5-a18c48e5f516"
-					(reference "#PWR045")
+					(reference "#PWR010")
 					(unit 1)
 				)
@@
 		(dnp no)
 		(fields_autoplaced yes)
-		(property "Reference" "#PWR02"
+		(property "Reference" "#PWR01"
 			(at 48.26 72.39 0)
 			(hide yes)
@@
 			(project "slapdaq-board"
 				(path "/13b31ec5-9d44-45c3-b3e5-a18c48e5f516"
-					(reference "#PWR02")
+					(reference "#PWR01")
 					(unit 1)
 				)
@@
 		(dnp no)
 		(fields_autoplaced yes)
-		(property "Reference" "#PWR01"
+		(property "Reference" "#PWR04"
 			(at 85.09 82.55 0)
 			(hide yes)
@@
 			(project "slapdaq-board"
 				(path "/13b31ec5-9d44-45c3-b3e5-a18c48e5f516"
-					(reference "#PWR01")
+					(reference "#PWR04")
 					(unit 1)
 				)
@@
 		(dnp no)
 		(fields_autoplaced yes)
-		(property "Reference" "#PWR05"
+		(property "Reference" "#PWR08"
 			(at 120.65 66.04 0)
 			(hide yes)
@@
 			(project "slapdaq-board"
 				(path "/13b31ec5-9d44-45c3-b3e5-a18c48e5f516"
-					(reference "#PWR05")
+					(reference "#PWR08")
 					(unit 1)
 				)
@@
 		(dnp no)
 		(fields_autoplaced yes)
-		(property "Reference" "D4"
+		(property "Reference" "D1"
 			(at 106.68 72.0724 90)
 			(show_name no)
@@
 			(project "slapdaq-board"
 				(path "/13b31ec5-9d44-45c3-b3e5-a18c48e5f516"
-					(reference "D4")
+					(reference "D1")
 					(unit 1)
 				)
@@
 		(dnp no)
 		(fields_autoplaced yes)
-		(property "Reference" "#PWR038"
+		(property "Reference" "#PWR011"
 			(at 120.65 124.46 0)
 			(hide yes)
@@
 			(project "slapdaq-board"
 				(path "/13b31ec5-9d44-45c3-b3e5-a18c48e5f516"
-					(reference "#PWR038")
+					(reference "#PWR011")
 					(unit 1)
 				)
@@
 		(in_pos_files yes)
 		(dnp no)
-		(property "Reference" "C29"
+		(property "Reference" "C4"
 			(at 102.87 95.25 90)
 			(show_name no)
@@
 			(project "slapdaq-board"
 				(path "/13b31ec5-9d44-45c3-b3e5-a18c48e5f516"
-					(reference "C29")
+					(reference "C4")
 					(unit 1)
 				)
@@
 		(dnp no)
 		(fields_autoplaced yes)
-		(property "Reference" "C2"
+		(property "Reference" "C5"
 			(at 124.46 74.0409 0)
 			(show_name no)
@@
 			(project "slapdaq-board"
 				(path "/13b31ec5-9d44-45c3-b3e5-a18c48e5f516"
-					(reference "C2")
+					(reference "C5")
 					(unit 1)
 				)
@@
 		(dnp no)
 		(fields_autoplaced yes)
-		(property "Reference" "D5"
+		(property "Reference" "D2"
 			(at 106.68 111.4424 90)
 			(show_name no)
@@
 			(project "slapdaq-board"
 				(path "/13b31ec5-9d44-45c3-b3e5-a18c48e5f516"
-					(reference "D5")
-					(unit 1)
-				)
+					(reference "D2")
+					(unit 1)
+				)

Commit message: 9/20/2026 schematic work
Parts:
- added D1, D2: BAT60A, Diode_SMD:D_SOD-323, symbol Diode:BAT60A
- added NT1: NetTie_2, symbol Device:NetTie_2
- added Q1: BSS84, Package_TO_SOT_SMD:SOT-23, symbol Transistor_FET:BSS84
- added R1, R2: 10k, Resistor_SMD:R_1206_3216Metric_Pad1.30x1.75mm_HandSolder, symbol Device:R
- C1, C2: footprint (none) -> Capacitor_Tantalum_SMD:CP_EIA-7260-38_AVX-R_HandSolder; MPN (none) -> 594D107X9025R2T; Mouser Link (none) -> https://www.mouser.com/en/ProductDetail/Vishay-Sprague/594D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
- C3, C4: footprint (none) -> Capacitor_SMD:C_1206_3216Metric_Pad1.33x1.80mm_HandSolder; MPN (none) -> GRM31CR73A103KW03L; Mouser Link (none) -> https://www.mouser.com/en/ProductDetail/Murata-Electronics/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
- C5: footprint (none) -> Capacitor_Tantalum_SMD:CP_EIA-7132-28_AVX-C_HandSolder; MPN 595D686X9010C2T -> 594D686X9010C2T; Mouser Link (none) -> https://www.mouser.com/en/ProductDetail/Vishay-Sprague/594D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
- C6: footprint (none) -> Capacitor_Tantalum_SMD:CP_EIA-7132-28_AVX-C_HandSolder; MPN 595D686X9010C2T -> 594D107X9016C2T; Mouser Link (none) -> https://www.mouser.com/en/ProductDetail/Vishay-Sprague/594D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
- D3: renamed from D1; footprint (none) -> Diode_SMD:D_SMA_Handsoldering; Mouser Link (none) -> https://www.mouser.com/en/ProductDetail/Diotec-Semiconducto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
- D4: renamed from D2; footprint (none) -> Diode_SMD:D_SMA_Handsoldering; Mouser Link (none) -> https://www.mouser.com/en/ProductDetail/Diotec-Semiconducto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
- F1: value 1A SLOW-BLOW -> 1.5A SLOW-BLOW; footprint Fuse:Fuse_1206_3216Metric -> Fuse:Fuse_1206_3216Metric_Pad1.42x1.75mm_HandSolder; MPN 0685T1000-01 -> SF-1206S150M-2; Mouser Link (none) -> https://www.mouser.com/en/ProductDetail/Bourns/SF-1206S150M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
- J1: value 12-24V POWER IN -> 12V POWER IN; footprint TerminalBlock_Phoenix:TerminalBlock_Phoenix_MKDS-1,5-2-5.08_1x02_P5.08mm_Horizontal -> (none); MPN 1715721 -> (none)
- L1: footprint (none) -> Inductor_SMD:L_Fastron_PISN_Handsoldering; MPN (none) -> DO3316P-473MLD; Mouser Link (none) -> https://www.mouser.com/en/ProductDetail/Coilcraft/DO3316P-4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
- L2: footprint (none) -> Inductor_SMD:L_Fastron_PISN_Handsoldering; MPN (none) -> DO3316P-683MLD; Mouser Link (none) -> https://www.mouser.com/en/ProductDetail/Coilcraft/DO3316P-6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
- U1: MPN LM2675M-3.3/NOPB -> LM2675MX-3.3/NOPB; Mouser Link (none) -> https://www.mouser.com/en/ProductDetail/Texas-Instruments/L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
- U2: MPN (none) -> LM2675MX-5.0/NOPB; Mouser Link (none) -> https://www.mouser.com/en/ProductDetail/Texas-Instruments/L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
Connections:
- net +3.3V: now also U1.4 (FB), Q1.2 (S)
- net +5V: now also U2.4 (FB), NT1.1
- net GND: now also R1.2, R2.2
- net Vbus: now also D2.2 (A), NT1.2, Q1.1 (G), R1.1
- net at C1.1, C2.1, U1.7 (VIN)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: now also D1.1 (K), D2.1 (K); no longer F1.2, U1.5 (ON/~{OFF}), U2.5 (ON/~{OFF})
- net at C3.2, D3.1 (K), L1.1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: no longer U1.4 (FB)
- net at C4.2, D4.1 (K), L2.1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: no longer U2.4 (FB)
- new net: Q1.3 (D), R2.1, U2.5 (ON/~{OFF})
- new net: D1.2 (A), F1.2
- no-connect marks 0 -> 1
Other:
- note added: "+5V is provided by USB when connected."
- note added: "Add screw terminal symbols here."
- note added: "For the 12 V and USB power supplies: 12 V only: both regulators on USB only: 3.3 V on and 5 V off. +5V net = Vbus Both: 3.3 V on and 5 V off. +5V net = Vbus"
- note added: "Turn off 5 V regulator when USB is connected."
- note removed: "For Grayson: Connect Vbus to the input of the 3.3 V regulator (and the +5V net?) I think that will allow the entire device to work with only USB power. Use schottky diodes."
- title: Power -> SlapDAQ - Power
- moved on the sheet: C1, C2, C3, C4, C5, C6, D3, D4, F1, J1, L1, L2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
