File: slapdaq-board.kicad_pcb (KiCad board)
At the start: 4 copper layers, 88 x 136 mm, 74 parts, among them J1 Higher Screw Terminals, J2 Lower Screw Terminals, J3 USB-C, Q1 BSS84, U1 LM2675M-3.3, U2 LM2675M-5, U3 ESP32-S3, U4 DT1042-04SO-7, U5 REF3333, U6 ADS1261, U7 MAX31856

Commit message: added logo to silkscreen
Parts:
- added G***: LOGO, LOGO, F.Cu at (168.8, 86.6)

Commit message: Finish rev. 1 PCB
Parts:
- C22: moved to B.Cu
- moved G*** 29.7 mm to (140.5, 95.5), turned to 0 degrees
- moved Q1 16.9 mm to (150.3, 174.0)
- moved R2 12.2 mm to (153.8, 177.5), turned to -90 degrees
- moved NT1 10.6 mm to (149.0, 167.2), turned to -45 degrees
- moved C22 10.1 mm to (135.5, 167.0), turned to 0 degrees
- moved R1 8.70 mm to (145.8, 176.5), turned to -90 degrees
- moved C21 7.30 mm to (141.5, 168.5)
- moved C20 6.37 mm to (138.0, 168.5)
- moved D2 3.84 mm to (134.8, 184.2), turned to 90 degrees
- moved R5 3.74 mm to (105.8, 95.5)
- moved R4 3.64 mm to (105.8, 104.2)
- moved C24 2.13 mm to (140.5, 153.9)
- moved C6 1.87 mm to (175.0, 153.0)
- moved C5 1.80 mm to (174.9, 120.0)
- moved C17 0.84 mm to (135.4, 173.6)
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Routing:
- net Net-(D1-K): track 2.75 -> 38.4 mm
- net Net-(Q1-D): track 8.72 -> 27.9 mm, vias 0 -> 2
- net Net-(U6-CAPP): track 18.4 -> 4.35 mm, vias 2 -> 1
- net GND: track 114.0 -> 103.2 mm, vias 43 -> 71
- net Net-(U6-CAPN): track 10.9 -> 5.14 mm, vias 2 -> 1
- net +3.3V: track 45.4 -> 40.7 mm, vias 23 -> 24
- net Net-(D6-A): track 8.28 -> 4.52 mm
- net Net-(D5-A): track 8.30 -> 4.66 mm
- net Net-(U5-OUT): track 13.7 -> 16.3 mm
- net +5V: track 60.5 -> 62.6 mm, vias 0 -> 2
- net SPI_Q: track 122.4 -> 120.4 mm
- net Net-(U6-AIN2): track 32.3 -> 33.8 mm
- net /MCU/WIFI_LED: track 39.5 -> 38.1 mm
- net Net-(U6-AIN3): track 29.2 -> 30.6 mm
- net Net-(U7-T+): track 31.0 -> 32.1 mm
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Other:
- board text added: "AC1"
- board text added: "AC2"
- board text added: "AV1"
- board text added: "AV2"
- board text added: "AV3"
- board text added: "AV4"
- board text added: "All dimensions in mm"
- board text added: "DIO0"
- board text added: "DIO1"
- board text added: "DIO2"
- board text added: "DIO3"
- board text added: "DIO4"
- board text added: "DIO5"
- board text added: "DIO6"
- board text added: "DIO7"
- board text added: "DV+"
- board text added: "DV-"
- board text added: "GND"
- board text added: "Grayson Riffe Leila Allebe Mia Gonzalez Senmache Kegan Dunn 10/12/2026 Rev. 1"
- board text added: "TH+"
- board text added: "TH-"
- board text added: "VCC"
